Commit message: refactor urdf.xacro of zu5 for composite

File: jaka_description/urdf/jaka_zu5.urdf.xacro (robot description, xacro)
@@ -1,467 +1,5 @@
-<?xml version="1.0" encoding="utf-8"?>
-<!-- This URDF was automatically created by SolidWorks to URDF Exporter! Originally created by Stephen Brawner (brawner@gmail.com)
-     Commit Version: 1.5.1-0-g916b5db  Build Version: 1.5.7152.31018
-     For more information, please see http://wiki.ros.org/sw_urdf_exporter -->
-<robot
-  name="jaka_zu5">
-  <!-- LINK -->
-  <link name="world" />
-  <link
-    name="Link_0">
-    <inertial>
-      <origin
-        xyz="0.00096371 8.8222E-08 0.019555"
-        rpy="0 0 0" />
-      <mass
-        value="4.0392" />
-      <inertia
-        ixx="0.0048763"
-        ixy="-1.8056E-07"
-        ixz="2.5196E-05"
-        iyy="0.0068003"
-        iyz="-1.7678E-09"
-        izz="0.010618" />
-    </inertial>
-    <visual>
-      <origin
-        xyz="0 0 0"
-        rpy="0 0 0" />
-      <geometry>
-        <mesh
-          filename="package://jaka_description/meshes/jaka_zu5_meshes/Link_0.STL" />
-      </geometry>
-      <material
-        name="">
-        <color
-          rgba="0.84706 0.84706 0.84706 1" />
-      </material>
-    </visual>
-    <collision>
-      <origin
-        xyz="0 0 0"
-        rpy="0 0 0" />
-      <geometry>
-        <mesh
-          filename="package://jaka_description/meshes/jaka_zu5_meshes/Link_0.STL" />
-      </geometry>
-    </collision>
-  </link>
-  <link
-    name="Link_1">
-    <inertial>
-      <origin
-        xyz="-2.5186E-07 0.0033226 -0.001509"
-        rpy="0 0 0" />
-      <mass
-        value="15.135" />
-      <inertia
-        ixx="0.044302"
-        ixy="1.5349E-07"
-        ixz="-6.1966E-07"
-        iyy="0.043091"
-        iyz="1.4326E-05"
-        izz="0.030523" />
-    </inertial>
-    <visual>
-      <origin
-        xyz="0 0 0"
-        rpy="0 0 0" />
-      <geometry>
-        <mesh
-          filename="package://jaka_description/meshes/jaka_zu5_meshes/Link_1.STL" />
-      </geometry>
-      <material
-        name="">
-        <color
-          rgba="0.84706 0.84706 0.84706 1" />
-      </material>
-    </visual>
-    <collision>
-      <origin
-        xyz="0 0 0"
-        rpy="0 0 0" />
-      <geometry>
-        <mesh
-          filename="package://jaka_description/meshes/jaka_zu5_meshes/Link_1.STL" />
-      </geometry>
-    </collision>
-  </link>
-  <link
-    name="Link_2">
-    <inertial>
-      <origin
-        xyz="0.215 6.4325E-09 -0.14315"
-        rpy="0 0 0" />
-      <mass
-        value="45.847" />
-      <inertia
-        ixx="0.10377"
-        ixy="-1.3562E-06"
-        ixz="2.544E-07"
-        iyy="1.5964"
-        iyz="2.1509E-08"
-        izz="1.5689" />
-    </inertial>
-    <visual>
-      <origin
-        xyz="0 0 0"
-        rpy="0 0 0" />
-      <geometry>
-        <mesh
-          filename="package://jaka_description/meshes/jaka_zu5_meshes/Link_2.STL" />
-      </geometry>
-      <material
-        name="">
-        <color
-          rgba="0.84706 0.84706 0.84706 1" />
-      </material>
-    </visual>
-    <collision>
-      <origin
-        xyz="0 0 0"
-        rpy="0 0 0" />
-      <geometry>
-        <mesh
-          filename="package://jaka_description/meshes/jaka_zu5_meshes/Link_2.STL" />
-      </geometry>
-    </collision>
-  </link>
-  <link
-    name="Link_3">
-    <inertial>
-      <origin
-        xyz="0.19087 -1.1862E-05 -0.010587"
-        rpy="0 0 0" />
-      <mass
-        value="18.069" />
-      <inertia
-        ixx="0.022066"
-        ixy="-3.4554E-06"
-        ixz="-0.022609"
-        iyy="0.41632"
-        iyz="1.1508E-08"
-        izz="0.41071" />
-    </inertial>
-    <visual>
-      <origin
-        xyz="0 0 0"
-        rpy="0 0 0" />
-      <geometry>
-        <mesh
-          filename="package://jaka_description/meshes/jaka_zu5_meshes/Link_3.STL" />
-      </geometry>
-      <material
-        name="">
-        <color
-          rgba="0.84706 0.84706 0.84706 1" />
-      </material>
-    </visual>
-    <collision>
-      <origin
-        xyz="0 0 0"
-        rpy="0 0 0" />
-      <geometry>
-        <mesh
-          filename="package://jaka_description/meshes/jaka_zu5_meshes/Link_3.STL" />
-      </geometry>
-    </collision>
-  </link>
-  <link
-    name="Link_4">
-    <inertial>
-      <origin
-        xyz="-2.1345E-06 -0.0058004 0.0026717"
-        rpy="0 0 0" />
-      <mass
-        value="5.5525" />
-      <inertia
-        ixx="0.0092564"
-        ixy="1.1341E-07"
-        ixz="-1.2578E-08"
-        iyy="0.0052251"
-        iyz="-8.3499E-05"
-        izz="0.0089683" />
-    </inertial>
-    <visual>
-      <origin
-        xyz="0 0 0"
-        rpy="0 0 0" />
-      <geometry>
-        <mesh
-          filename="package://jaka_description/meshes/jaka_zu5_meshes/Link_4.STL" />
-      </geometry>
-      <material
-        name="">
-        <color
-          rgba="0.84706 0.84706 0.84706 1" />
-      </material>
-    </visual>
-    <collision>
-      <origin
-        xyz="0 0 0"
-        rpy="0 0 0" />
-      <geometry>
-        <mesh
-          filename="package://jaka_description/meshes/jaka_zu5_meshes/Link_4.STL" />
-      </geometry>
-    </collision>
-  </link>
-  <link
-    name="Link_5">
-    <inertial>
-      <origin
-        xyz="-2.0304E-06 -0.0028889 -0.0023424"
-        rpy="0 0 0" />
-      <mass
-        value="6.3339" />
-      <inertia
-        ixx="0.012993"
-        ixy="-1.0764E-07"
-        ixz="5.8559E-09"
-        iyy="0.0058454"
-        iyz="4.5426E-05"
-        izz="0.0127" />
-    </inertial>
-    <visual>
-      <origin
-        xyz="0 0 0"
-        rpy="0 0 0" />
-      <geometry>
-        <mesh
-          filename="package://jaka_description/meshes/jaka_zu5_meshes/Link_5.STL" />
-      </geometry>
-      <material
-        name="">
-        <color
-          rgba="0.84706 0.84706 0.84706 1" />
-      </material>
-    </visual>
-    <collision>
-      <origin
-        xyz="0 0 0"
-        rpy="0 0 0" />
-      <geometry>
-        <mesh
-          filename="package://jaka_description/meshes/jaka_zu5_meshes/Link_5.STL" />
-      </geometry>
-    </collision>
-  </link>
-  <link
-    name="Link_6">
-    <inertial>
-      <origin
-        xyz="2.7652E-05 -1.3485E-05 -0.021245"
-        rpy="0 0 0" />
-      <mass
-        value="1.4169" />
-      <inertia
-        ixx="0.00071853"
-        ixy="-6.9778E-07"
-        ixz="-6.378E-07"
-        iyy="0.00072375"
-        iyz="8.3072E-07"
-        izz="0.0011337" />
-    </inertial>
-    <visual>
-      <origin
-        xyz="0 0 0"
-        rpy="0 0 0" />
-      <geometry>
-        <mesh
-          filename="package://jaka_description/meshes/jaka_zu5_meshes/Link_6.STL" />
-      </geometry>
-      <material
-        name="">
-        <color
-          rgba="0.84706 0.84706 0.84706 1" />
-      </material>
-    </visual>
-    <collision>
-      <origin
-        xyz="0 0 0"
-        rpy="0 0 0" />
-      <geometry>
-        <mesh
-          filename="package://jaka_description/meshes/jaka_zu5_meshes/Link_6.STL" />
-      </geometry>
-    </collision>
-  </link>
-  <!-- JOINT -->
-  <joint name="fixed" type="fixed">
-     <parent link="world"/>
-     <child link="Link_0"/>
-  </joint>
-  <joint
-    name="joint_1"
-    type="revolute">
-    <origin
-      xyz="0 0 0.12015"
-      rpy="0 0 0" />
-    <parent
-      link="Link_0" />
-    <child
-      link="Link_1" />
-    <axis
-      xyz="0 0 1" />
-    <limit
-      lower="-6.28"
-      upper="6.28"
-      effort="2000"
-      velocity="1.57" />
-  </joint>
-  <joint
-    name="joint_2"
-    type="revolute">
-    <origin
-      xyz="0 0 0"
-      rpy="1.5708 0 0" />
-    <parent
-      link="Link_1" />
-    <child
-      link="Link_2" />
-    <axis
-      xyz="0 0 1" />
-    <limit
-      lower="-1.48"
-      upper="4.62"
-      effort="5000"
-      velocity="1.57" />
-  </joint>
-  <joint
-    name="joint_3"
-    type="revolute">
-    <origin
-      xyz="0.43 0 0"
-      rpy="0 0 0" />
-    <parent
-      link="Link_2" />
-    <child
-      link="Link_3" />
-    <axis
-      xyz="0 0 1" />
-    <limit
-      lower="-3.05"
-      upper="3.05"
-      effort="5000"
-      velocity="1.57" />
-  </joint>
-  <joint
-    name="joint_4"
-    type="revolute">
-    <origin
-      xyz="0.3685 -1.185E-05 -0.114"
-      rpy="0 0 0" />
-    <parent
-      link="Link_3" />
-    <child
-      link="Link_4" />
-    <axis
-      xyz="0 0 1" />
-    <limit
-      lower="-1.48"
-      upper="4.62"
-      effort="2000"
-      velocity="1.57" />
-  </joint>
-  <joint
-    name="joint_5"
-    type="revolute">
-    <origin
-      xyz="0 -0.1135 0"
-      rpy="1.5708 0 0" />
-    <parent
-      link="Link_4" />
-    <child
-      link="Link_5" />
-    <axis
-      xyz="0 0 1" />
-    <limit
-      lower="-6.28"
-      upper="6.28"
-      effort="3000"
-      velocity="1.57" />
-  </joint>
-  <joint
-    name="joint_6"
-    type="revolute">
-    <origin
-      xyz="0 0.107 0"
-      rpy="-1.5708 0 0" />
-    <parent
-      link="Link_5" />
-    <child
-      link="Link_6" />
-    <axis
-      xyz="0 0 1" />
-    <limit
-      lower="-6.28"
-      upper="6.28"
-      effort="1000"
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