Commit message: synchronized with jaka official repo

File: jaka_description/urdf/jaka_Pro 7.urdf (robot description, URDF)
Before this commit: robot jaka_zu5, 8 links, 7 joints
Links:
- removed link Link_0
- added link base_link, mass 0.57896; collision mesh filename=package://jaka_description/meshes/jaka_pro7_meshes/base_lin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; visual mesh filename=package://jaka_description/meshes/jaka_pro7_meshes/base_lin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
- link Link_1: mass 15.135 -> 1.9271; geometry collision mesh filename=package://jaka_description/meshes/jaka_pro7_meshes/Link_01.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; visual mesh filename=package://jaka_description/meshes/jaka_pro7_meshes/Link_01.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
- link Link_2: mass 45.847 -> 5.4599; geometry collision mesh filename=package://jaka_description/meshes/jaka_pro7_meshes/Link_02.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; visual mesh filename=package://jaka_description/meshes/jaka_pro7_meshes/Link_02.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
- link Link_3: mass 18.069 -> 2.1077; geometry collision mesh filename=package://jaka_description/meshes/jaka_pro7_meshes/Link_03.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; visual mesh filename=package://jaka_description/meshes/jaka_pro7_meshes/Link_03.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
- link Link_4: mass 5.5525 -> 0.70529; geometry collision mesh filename=package://jaka_description/meshes/jaka_pro7_meshes/Link_04.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; visual mesh filename=package://jaka_description/meshes/jaka_pro7_meshes/Link_04.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
- link Link_5: mass 6.3339 -> 0.80153; geometry collision mesh filename=package://jaka_description/meshes/jaka_pro7_meshes/Link_05.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; visual mesh filename=package://jaka_description/meshes/jaka_pro7_meshes/Link_05.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
- link Link_6: mass 1.4169 -> 0.17604; geometry collision mesh filename=package://jaka_description/meshes/jaka_pro7_meshes/Link_06.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; visual mesh filename=package://jaka_description/meshes/jaka_pro7_meshes/Link_06.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
Joints:
- joint fixed: child Link_0 -> base_link
- joint joint_1: parent Link_0 -> base_link
- joint joint_2: limit lower=-1.48 upper=4.62 effort=5000 velocity=1.57 -> lower=-1.48 upper=4.62 effort=8000 velocity=1.57
- joint joint_3: limit lower=-3.05 upper=3.05 effort=5000 velocity=1.57 -> lower=-3.05 upper=3.05 effort=8000 velocity=1.57; origin xyz=0.43 0 0 rpy=0 0 0 -> xyz=0.36 0 0 rpy=0 0 0
- joint joint_4: origin xyz=0.3685 -1.185E-05 -0.114 rpy=0 0 0 -> xyz=0.3035 0 -0.11502 rpy=0 0 0

File: jaka_description/urdf/jaka_a5.urdf (robot description, URDF)
Before this commit: robot jaka_zu5, 8 links, 7 joints
Links:
- removed link Link_0
- removed link Link_1
- removed link Link_2
- removed link Link_3
- removed link Link_4
- removed link Link_5
- removed link Link_6
- added link J1, mass 15.135; collision mesh filename=package://jaka_description/meshes/jaka_a5_meshes/J1.STL; visual mesh filename=package://jaka_description/meshes/jaka_a5_meshes/J1.STL
- added link J2, mass 5.7891; collision mesh filename=package://jaka_description/meshes/jaka_a5_meshes/J2.STL; visual mesh filename=package://jaka_description/meshes/jaka_a5_meshes/J2.STL
- added link J3, mass 2.5808; collision mesh filename=package://jaka_description/meshes/jaka_a5_meshes/J3.STL; visual mesh filename=package://jaka_description/meshes/jaka_a5_meshes/J3.STL
- added link J4, mass 5.5377; collision mesh filename=package://jaka_description/meshes/jaka_a5_meshes/J4.STL; visual mesh filename=package://jaka_description/meshes/jaka_a5_meshes/J4.STL
- added link J5, mass 0.81207; collision mesh filename=package://jaka_description/meshes/jaka_a5_meshes/J5.STL; visual mesh filename=package://jaka_description/meshes/jaka_a5_meshes/J5.STL
- added link J6, mass 1.336; collision mesh filename=package://jaka_description/meshes/jaka_a5_meshes/J6.STL; visual mesh filename=package://jaka_description/meshes/jaka_a5_meshes/J6.STL
- added link base_link, mass 0.52663; collision mesh filename=package://jaka_description/meshes/jaka_a5_meshes/base_link.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; visual mesh filename=package://jaka_description/meshes/jaka_a5_meshes/base_link.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
Joints:
- joint fixed: child Link_0 -> base_link
- joint joint_1: child Link_1 -> J1; origin xyz=0 0 0.12015 rpy=0 0 0 -> xyz=0 -0.00022535 0.12015 rpy=0 0 0; parent Link_0 -> base_link
- joint joint_2: child Link_2 -> J2; parent Link_1 -> J1
- joint joint_3: child Link_3 -> J3; parent Link_2 -> J2
- joint joint_4: child Link_4 -> J4; origin xyz=0.3685 -1.185E-05 -0.114 rpy=0 0 0 -> xyz=0.3685 0 -0.115 rpy=0 0 0; parent Link_3 -> J3
- joint joint_5: child Link_5 -> J5; origin xyz=0 -0.1135 0 rpy=1.5708 0 0 -> xyz=0 -0.1135 0 rpy=1.5708 -0.00010901 0; parent Link_4 -> J4
- joint joint_6: axis 0 0 1 -> -0.00010901 0 1; child Link_6 -> J6; origin xyz=0 0.107 0 rpy=-1.5708 0 0 -> xyz=0 0.107 0 rpy=-1.5708 0 -0.00010901; parent Link_5 -> J5
