Commit message: synchronized from jaka official

File: jaka_description/urdf/jaka_a12.urdf (robot description, URDF)
Before this commit: robot jaka_a12, 8 links, 7 joints
Joints:
- joint joint_1: limit lower=-6.28 upper=6.28 effort=2000 velocity=1.57 -> lower=-6.28 upper=6.28 effort=2000 velocity=2.62; origin xyz=-9.3823E-05 0 0.14265 rpy=0 0 0 -> xyz=9.3823E-05 0 0.14265 rpy=0 0 0
- joint joint_2: limit lower=-1.48 upper=4.62 effort=8000 velocity=1.57 -> lower=-6.28 upper=6.28 effort=8000 velocity=2.62
- joint joint_3: limit lower=-3.05 upper=3.05 effort=8000 velocity=1.57 -> lower=-6.28 upper=6.28 effort=8000 velocity=3.67
- joint joint_4: limit lower=-1.48 upper=4.62 effort=2000 velocity=1.57 -> lower=-6.28 upper=6.28 effort=2000 velocity=3.67
- joint joint_5: limit lower=-6.28 upper=6.28 effort=3000 velocity=1.57 -> lower=-6.28 upper=6.28 effort=3000 velocity=3.67
- joint joint_6: limit lower=-6.28 upper=6.28 effort=1000 velocity=1.57 -> lower=-6.28 upper=6.28 effort=1000 velocity=3.67

File: jaka_description/urdf/jaka_a5.urdf (robot description, URDF)
Before this commit: robot jaka_a5, 8 links, 7 joints
Joints:
- joint joint_1: limit lower=-6.28 upper=6.28 effort=2000 velocity=1.57 -> lower=-6.28 upper=6.28 effort=2000 velocity=3.665
- joint joint_2: limit lower=-1.48 upper=4.62 effort=5000 velocity=1.57 -> lower=-1.48 upper=4.628 effort=5000 velocity=3.665
- joint joint_3: limit lower=-3.05 upper=3.05 effort=5000 velocity=1.57 -> lower=-3.05 upper=3.05 effort=5000 velocity=3.665
- joint joint_4: limit lower=-1.48 upper=4.62 effort=2000 velocity=1.57 -> lower=-1.48 upper=4.62 effort=2000 velocity=3.665
- joint joint_5: limit lower=-6.28 upper=6.28 effort=3000 velocity=1.57 -> lower=-6.28 upper=6.28 effort=3000 velocity=3.665
- joint joint_6: limit lower=-6.28 upper=6.28 effort=1000 velocity=1.57 -> lower=-6.28 upper=6.28 effort=1000 velocity=3.665

File: jaka_description/urdf/jaka_zu5.xacro (robot description, xacro)
@@ -34,5 +34,5 @@
       <child link="${prefix}link_1"/>
       <axis xyz="0 0 1"/>
-      <limit lower="-6.28" upper="6.28" effort="2000" velocity="1.57" />
+      <limit lower="-6.28" upper="6.28" effort="2000" velocity="3.14" />
     </joint>
     <!--link2 to link1-->
@@ -46,5 +46,5 @@
       <child link="${prefix}link_2"/>
       <axis xyz="0 0 1"/>
-      <limit lower="-1.48" upper="4.62" effort="5000" velocity="1.57" />
+      <limit lower="-1.48" upper="4.62" effort="5000" velocity="3.14" />
     </joint>
     <!--link3 to link2-->
@@ -58,5 +58,5 @@
       <child link="${prefix}link_3"/>
       <axis xyz="0 0 1"/>
-      <limit lower="-3.05" upper="3.05" effort="5000" velocity="1.57"/>
+      <limit lower="-3.05" upper="3.05" effort="5000" velocity="3.14"/>
     </joint>
     <!--link4 to link3-->
@@ -70,5 +70,5 @@
       <child link="${prefix}link_4"/>
       <axis xyz="0 0 1"/>
-      <limit lower="-1.48" upper="4.62" effort="2000" velocity="1.57" />
+      <limit lower="-1.48" upper="4.62" effort="2000" velocity="3.14" />
     </joint>
     <!--link5 to link4-->
@@ -82,5 +82,5 @@
       <child link="${prefix}link_5"/>
       <axis xyz="0 0 1"/>
-      <limit lower="-6.28" upper="6.28" effort="3000" velocity="1.57"/>
+      <limit lower="-6.28" upper="6.28" effort="3000" velocity="3.14"/>
     </joint>
     <!--link6 to link5-->
@@ -94,5 +94,5 @@
       <child link="${prefix}link_6"/>
       <axis xyz="0 0 1"/>
-      <limit lower="-6.28" upper="6.28" effort="1000" velocity="1.57"/>
+      <limit lower="-6.28" upper="6.28" effort="1000" velocity="3.14"/>
     </joint>
   </xacro:macro>
