Commit message: revise moveit_config for a5

File: jaka_description/urdf/jaka_a5.urdf (robot description, URDF)
Before this commit: robot jaka_a5, 8 links, 7 joints
Links:
- removed link base_link
- added link Link_0, mass 0.52663; collision mesh filename=package://jaka_description/meshes/jaka_a5_meshes/Link_0.STL; visual mesh filename=package://jaka_description/meshes/jaka_a5_meshes/Link_0.STL
Joints:
- joint fixed: child base_link -> Link_0
- joint joint_1: parent base_link -> Link_0

File: jaka_description/urdf/jaka_a5.xacro (robot description, xacro)
@@ -1,7 +1,7 @@
 <?xml version='1.0' encoding='utf-8'?>
-<robot name="jaka_zu5" xmlns:xacro="http://www.ros.org/wiki/xacro">
+<robot name="jaka_a5" xmlns:xacro="http://www.ros.org/wiki/xacro">
   <xacro:macro name="jaka_arm" params="connected_to:='' prefix:='' xyz=:'0 0 0' rpy=:'0 0 0' gazebo:=false">
     <xacro:include filename="$(find jaka_description)/urdf/components.xacro"/>
-    <xacro:property name="mesh_path" value="jaka_description/meshes/jaka_zu5_meshes"/>
+    <xacro:property name="mesh_path" value="jaka_description/meshes/jaka_a5_meshes"/>
     <xacro:unless value="${not connected_to}">
       <joint name="joint_${connected_to}" type="fixed">
@@ -21,23 +21,23 @@
     <!--link0 to world-->
     <xacro:link_arm name="0" prefix="${prefix}"
-      ixyz="0.00096371 8.8222E-08 0.019555" ixx="0.0048763" ixy="-1.8056E-07" ixz="2.5196E-05" iyy="0.0068003" iyz="-1.7678E-09" izz="0.010618" mass="4.0392"
-      rgba="0.84706 0.84706 0.84706 1" stl_path="package://${mesh_path}/Link_0.STL" gazebo="${gazebo}">
+      ixyz="0.0028167 -0.00019454 0.019544" ixx="0.0006297" ixy="6.7091E-08" ixz="3.4682E-06" iyy="0.00095727" iyz="2.4476E-07" izz="0.0014514" mass="0.52663"
+      rgba="0.86667 0.86667 0.8902 1" stl_path="package://${mesh_path}/Link_0.STL" gazebo="${gazebo}">
     </xacro:link_arm>
     <!--link1 to link0-->
     <xacro:link_arm name="1" prefix="${prefix}"
       ixyz="-2.5186E-07 0.0033226 -0.001509" ixx="0.044302" ixy="1.5349E-07" ixz="-6.1966E-07" iyy="0.043091" iyz="1.4326E-05" izz="0.030523" mass="15.135"
-      rgba="0.84706 0.84706 0.84706 1" stl_path="package://${mesh_path}/Link_1.STL" gazebo="${gazebo}">
+      rgba="0.79216 0.81961 0.93333 1" stl_path="package://${mesh_path}/Link_1.STL" gazebo="${gazebo}">
     </xacro:link_arm>
     <joint name="${prefix}joint_1" type="revolute">
-      <origin xyz="0 0 0.12015" rpy="0 0 0"/>
+      <origin xyz="0 -0.00022535 0.12015" rpy="0 0 0"/>
       <parent link="${prefix}link_0"/>
       <child link="${prefix}link_1"/>
       <axis xyz="0 0 1"/>
-      <limit lower="-6.28" upper="6.28" effort="2000" velocity="3.14"/>
+      <limit lower="-6.28" upper="6.28" effort="2000" velocity="3.665"/>
     </joint>
     <!--link2 to link1-->
     <xacro:link_arm name="2" prefix="${prefix}"
-      ixyz="0.215 6.4325E-09 -0.14315" ixx="0.10377" ixy="-1.3562E-06" ixz="2.544E-07" iyy="1.5964" iyz="2.1509E-08" izz="1.5689" mass="45.847"
-      rgba="0.84706 0.84706 0.84706 1" stl_path="package://${mesh_path}/Link_2.STL" gazebo="${gazebo}">
+      ixyz="0.215 4.9016E-09 -0.14314" ixx="0.013095" ixy="-4.1856E-09" ixz="2.9241E-08" iyy="0.20279" iyz="2.1723E-09" izz="0.19928" mass="5.7891"
+      rgba="0.79216 0.81961 0.93333 1" stl_path="package://${mesh_path}/Link_2.STL" gazebo="${gazebo}">
     </xacro:link_arm>
     <joint name="${prefix}joint_2" type="revolute">
@@ -46,10 +46,10 @@
       <child link="${prefix}link_2"/>
       <axis xyz="0 0 1"/>
-      <limit lower="-1.48" upper="4.62" effort="5000" velocity="3.14"/>
+      <limit lower="-1.48" upper="4.628" effort="5000" velocity="3.665"/>
     </joint>
     <!--link3 to link2-->
     <xacro:link_arm name="3" prefix="${prefix}"
-      ixyz="0.19087 -1.1862E-05 -0.010587" ixx="0.022066" ixy="-3.4554E-06" ixz="-0.022609" iyy="0.41632" iyz="1.1508E-08" izz="0.41071" mass="18.069"
-      rgba="0.84706 0.84706 0.84706 1" stl_path="package://${mesh_path}/Link_3.STL" gazebo="${gazebo}">
+      ixyz="0.17601 -7.8489E-07 -0.0097984" ixx="0.0032112" ixy="1.1156E-07" ixz="-0.0022739" iyy="0.05921" iyz="3.3121E-08" izz="0.058511" mass="2.5808"
+      rgba="0.79216 0.81961 0.93333 1" stl_path="package://${mesh_path}/Link_3.STL" gazebo="${gazebo}">
     </xacro:link_arm>
     <joint name="${prefix}joint_3" type="revolute">
@@ -58,41 +58,41 @@
       <child link="${prefix}link_3"/>
       <axis xyz="0 0 1"/>
-      <limit lower="-3.05" upper="3.05" effort="5000" velocity="3.14"/>
+      <limit lower="-3.05" upper="3.05" effort="5000" velocity="3.665"/>
     </joint>
     <!--link4 to link3-->
     <xacro:link_arm name="4" prefix="${prefix}"
-      ixyz="-2.1345E-06 -0.0058004 0.0026717" ixx="0.0092564" ixy="1.1341E-07" ixz="-1.2578E-08" iyy="0.0052251" iyz="-8.3499E-05" izz="0.0089683" mass="5.5525"
+      ixyz="-2.1463E-06 -0.0059512 0.0026789" ixx="0.0092004" ixy="1.17E-07" ixz="-1.3683E-08" iyy="0.0052083" iyz="-8.5741E-05" izz="0.0089125" mass="5.5377"
       rgba="0.84706 0.84706 0.84706 1" stl_path="package://${mesh_path}/Link_4.STL" gazebo="${gazebo}">
     </xacro:link_arm>
     <joint name="${prefix}joint_4" type="revolute">
-      <origin xyz="0.3685 -1.185E-05 -0.114" rpy="0 0 0"/>
+      <origin xyz="0.3685 0 -0.115" rpy="0 0 0"/>
       <parent link="${prefix}link_3"/>
       <child link="${prefix}link_4"/>
       <axis xyz="0 0 1"/>
-      <limit lower="-1.48" upper="4.62" effort="2000" velocity="3.14"/>
+      <limit lower="-1.48" upper="4.62" effort="2000" velocity="3.665" />
     </joint>
     <!--link5 to link4-->
     <xacro:link_arm name="5" prefix="${prefix}"
-      ixyz="-2.0304E-06 -0.0028889 -0.0023424" ixx="0.012993" ixy="-1.0764E-07" ixz="5.8559E-09" iyy="0.0058454" iyz="4.5426E-05" izz="0.0127" mass="6.3339"
-      rgba="0.84706 0.84706 0.84706 1" stl_path="package://${mesh_path}/Link_5.STL" gazebo="${gazebo}">
+      ixyz="-2.2875E-08 -0.0015344 -0.0023275" ixx="0.0016825" ixy="2.829E-09" ixz="-1.1984E-08" iyy="0.00074766" iyz="3.2415E-06" izz="0.0016452" mass="0.81207"
+      rgba="0.79216 0.81961 0.93333 1" stl_path="package://${mesh_path}/Link_5.STL" gazebo="${gazebo}">
     </xacro:link_arm>
     <joint name="${prefix}joint_5" type="revolute">
-      <origin xyz="0 -0.1135 0" rpy="1.5708 0 0"/>
+      <origin xyz="0 -0.1135 0" rpy="1.5708 -0.00010901 0"/>
       <parent link="${prefix}link_4"/>
       <child link="${prefix}link_5"/>
       <axis xyz="0 0 1"/>
-      <limit lower="-6.28" upper="6.28" effort="3000" velocity="3.14"/>
+      <limit lower="-6.28" upper="6.28" effort="3000" velocity="3.665"/>
     </joint>
     <!--link6 to link5-->
     <xacro:link_arm name="6" prefix="${prefix}"
-      ixyz="2.7652E-05 -1.3485E-05 -0.021245" ixx="0.00071853" ixy="-6.9778E-07" ixz="-6.378E-07" iyy="0.00072375" iyz="8.3072E-07" izz="0.0011337" mass="1.4169"
+      ixyz="3.1532E-05 -1.4302E-05 -0.02023" ixx="0.00066124" ixy="-6.979E-07" ixz="-6.4232E-07" iyy="0.00066646" iyz="8.1119E-07" izz="0.0010673" mass="1.336"
       rgba="0.84706 0.84706 0.84706 1" stl_path="package://${mesh_path}/Link_6.STL" gazebo="${gazebo}">
     </xacro:link_arm>
     <joint name="${prefix}joint_6" type="revolute">
-      <origin xyz="0 0.107 0" rpy="-1.5708 0 0"/>
+      <origin xyz="0 0.107 0" rpy="-1.5708 0 -0.00010901"/>
       <parent link="${prefix}link_5"/>
       <child link="${prefix}link_6"/>
       <axis xyz="0 0 1"/>
-      <limit lower="-6.28" upper="6.28" effort="1000" velocity="3.14"/>
+      <limit lower="-6.28" upper="6.28" effort="1000" velocity="3.665"/>
     </joint>
   </xacro:macro>
